File: 18650_Charger/18650_Charger.kicad_sch (KiCad schematic)
At the start: 12 parts, among them J1 IN_5V, J2 IN_0V, J3 BAT_5V, J4 BAT_0V, U1 TP4056

Commit message: V3
Parts:
- R3: footprint LED_SMD:LED_0603_1608Metric -> LED_SMD:LED_0603_1608Metric_Pad1.05x0.95mm_HandSolder
Changed lines of the file:
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@@
 			)
 		)
-		(property "Footprint" "LED_SMD:LED_0603_1608Metric"
+		(property "Footprint" "LED_SMD:LED_0603_1608Metric_Pad1.05x0.95mm_HandSolder"
 			(at 129.032 85.09 90)
 			(effects
